File: kicad/UNL2803.sch (KiCad schematic (older format))
At the start: 19 parts, among them P15 CONN_01X08, P16 CONN_01X08, U4 ULN2803

Commit message: prototipo base para icaro version SMD
Parts:
- D10, D11, D12, D13, D6, D7, D8, D9: footprint LEDs:LED-5MM -> (none); symbol LED -> LED-RESCUE-np08
- P15: value CONN_01X08 -> PORTB; footprint Pin_Headers:Pin_Header_Straight_1x08 -> Pin_Headers:Pin_Header_Straight_1x08_Pitch1.27mm
- P16: footprint Pin_Headers:Pin_Header_Straight_1x08 -> (none)
- R10, R11, R12, R5, R6, R7, R8, R9: footprint Resistors_ThroughHole:Resistor_Horizontal_RM7mm -> (none)
- U4: footprint Housings_DIP:DIP-18_W7.62mm -> (none)
Changed lines of the file:
@@
 EESchema Schematic File Version 2
+LIBS:np08-rescue
 LIBS:power
 LIBS:device
@@
 F 0 "U4" H 5900 5750 60  0000 C CNN
 F 1 "ULN2803" H 5900 4750 60  0000 C CNN
-F 2 "Housings_DIP:DIP-18_W7.62mm" H 5650 5250 60  0001 C CNN
+F 2 "" H 5650 5250 60  0001 C CNN
 F 3 "" H 5650 5250 60  0000 C CNN
 	1    5650 5250
@@
 F 0 "R5" V 7330 3800 50  0000 C CNN
 F 1 "R" V 7250 3800 50  0000 C CNN
-F 2 "Resistors_ThroughHole:Resistor_Horizontal_RM7mm" V 7180 3800 50  0001 C CNN
+F 2 "" V 7180 3800 50  0001 C CNN
 F 3 "" H 7250 3800 50  0000 C CNN
 	1    7250 3800
@@
 F 0 "R9" V 7530 3900 50  0000 C CNN
 F 1 "R" V 7450 3900 50  0000 C CNN
-F 2 "Resistors_ThroughHole:Resistor_Horizontal_RM7mm" V 7380 3900 50  0001 C CNN
+F 2 "" V 7380 3900 50  0001 C CNN
 F 3 "" H 7450 3900 50  0000 C CNN
 	1    7450 3900
@@
 F 0 "R6" V 7330 4000 50  0000 C CNN
 F 1 "R" V 7250 4000 50  0000 C CNN
-F 2 "Resistors_ThroughHole:Resistor_Horizontal_RM7mm" V 7180 4000 50  0001 C CNN
+F 2 "" V 7180 4000 50  0001 C CNN
 F 3 "" H 7250 4000 50  0000 C CNN
 	1    7250 4000
@@
 F 0 "R10" V 7530 4100 50  0000 C CNN
 F 1 "R" V 7450 4100 50  0000 C CNN
-F 2 "Resistors_ThroughHole:Resistor_Horizontal_RM7mm" V 7380 4100 50  0001 C CNN
+F 2 "" V 7380 4100 50  0001 C CNN
 F 3 "" H 7450 4100 50  0000 C CNN
 	1    7450 4100
@@
 F 0 "R7" V 7330 4200 50  0000 C CNN
 F 1 "R" V 7250 4200 50  0000 C CNN
-F 2 "Resistors_ThroughHole:Resistor_Horizontal_RM7mm" V 7180 4200 50  0001 C CNN
+F 2 "" V 7180 4200 50  0001 C CNN
 F 3 "" H 7250 4200 50  0000 C CNN
 	1    7250 4200
@@
 F 0 "R11" V 7530 4300 50  0000 C CNN
 F 1 "R" V 7450 4300 50  0000 C CNN
-F 2 "Resistors_ThroughHole:Resistor_Horizontal_RM7mm" V 7380 4300 50  0001 C CNN
+F 2 "" V 7380 4300 50  0001 C CNN
 F 3 "" H 7450 4300 50  0000 C CNN
 	1    7450 4300
@@
 F 0 "R8" V 7330 4400 50  0000 C CNN
 F 1 "R" V 7250 4400 50  0000 C CNN
-F 2 "Resistors_ThroughHole:Resistor_Horizontal_RM7mm" V 7180 4400 50  0001 C CNN
+F 2 "" V 7180 4400 50  0001 C CNN
 F 3 "" H 7250 4400 50  0000 C CNN
 	1    7250 4400
@@
 F 0 "R12" V 7530 4500 50  0000 C CNN
 F 1 "R" V 7450 4500 50  0000 C CNN
-F 2 "Resistors_ThroughHole:Resistor_Horizontal_RM7mm" V 7380 4500 50  0001 C CNN
+F 2 "" V 7380 4500 50  0001 C CNN
 F 3 "" H 7450 4500 50  0000 C CNN
 	1    7450 4500
@@
 	7300 4500 6900 4500
 $Comp
-L LED D6
+L LED-RESCUE-np08 D6
 U 1 1 57A4DC0A
 P 7900 3800
+AR Path="/57A4DC0A" Ref="D6"  Part="1"
+AR Path="/57A4D8D4/57A4DC0A" Ref="D6"  Part="1"
 F 0 "D6" H 7900 3900 50  0000 C CNN
 F 1 "LED" H 7900 3700 50  0000 C CNN
-F 2 "LEDs:LED-5MM" H 7900 3800 50  0001 C CNN
+F 2 "" H 7900 3800 50  0001 C CNN
 F 3 "" H 7900 3800 50  0000 C CNN
 	1    7900 3800
@@
 $EndComp
 $Comp
-L LED D7
+L LED-RESCUE-np08 D7
 U 1 1 57A4DC4B
 P 8200 3900
+AR Path="/57A4DC4B" Ref="D7"  Part="1"
+AR Path="/57A4D8D4/57A4DC4B" Ref="D7"  Part="1"
 F 0 "D7" H 8200 4000 50  0000 C CNN
 F 1 "LED" H 8200 3800 50  0000 C CNN
-F 2 "LEDs:LED-5MM" H 8200 3900 50  0001 C CNN
+F 2 "" H 8200 3900 50  0001 C CNN
 F 3 "" H 8200 3900 50  0000 C CNN
 	1    8200 3900
@@
 $EndComp
 $Comp
-L LED D8
+L LED-RESCUE-np08 D8
 U 1 1 57A4DC8A
 P 8500 4000
+AR Path="/57A4DC8A" Ref="D8"  Part="1"
+AR Path="/57A4D8D4/57A4DC8A" Ref="D8"  Part="1"
 F 0 "D8" H 8500 4100 50  0000 C CNN
 F 1 "LED" H 8500 3900 50  0000 C CNN
-F 2 "LEDs:LED-5MM" H 8500 4000 50  0001 C CNN
+F 2 "" H 8500 4000 50  0001 C CNN
 F 3 "" H 8500 4000 50  0000 C CNN
 	1    8500 4000
@@
 $EndComp
 $Comp
-L LED D9
+L LED-RESCUE-np08 D9
 U 1 1 57A4DCFC
 P 8800 4100
+AR Path="/57A4DCFC" Ref="D9"  Part="1"
+AR Path="/57A4D8D4/57A4DCFC" Ref="D9"  Part="1"
 F 0 "D9" H 8800 4200 50  0000 C CNN
 F 1 "LED" H 8800 4000 50  0000 C CNN
-F 2 "LEDs:LED-5MM" H 8800 4100 50  0001 C CNN
+F 2 "" H 8800 4100 50  0001 C CNN
 F 3 "" H 8800 4100 50  0000 C CNN
 	1    8800 4100
@@
 $EndComp
 $Comp
-L LED D10
+L LED-RESCUE-np08 D10
 U 1 1 57A4DE04
 P 9100 4200
+AR Path="/57A4DE04" Ref="D10"  Part="1"
+AR Path="/57A4D8D4/57A4DE04" Ref="D10"  Part="1"
 F 0 "D10" H 9100 4300 50  0000 C CNN
 F 1 "LED" H 9100 4100 50  0000 C CNN
-F 2 "LEDs:LED-5MM" H 9100 4200 50  0001 C CNN
+F 2 "" H 9100 4200 50  0001 C CNN
 F 3 "" H 9100 4200 50  0000 C CNN
 	1    9100 4200
@@
 $EndComp
 $Comp
-L LED D11
+L LED-RESCUE-np08 D11
 U 1 1 57A4DE4E
 P 9400 4300
+AR Path="/57A4DE4E" Ref="D11"  Part="1"
+AR Path="/57A4D8D4/57A4DE4E" Ref="D11"  Part="1"
 F 0 "D11" H 9400 4400 50  0000 C CNN
 F 1 "LED" H 9400 4200 50  0000 C CNN
-F 2 "LEDs:LED-5MM" H 9400 4300 50  0001 C CNN
+F 2 "" H 9400 4300 50  0001 C CNN
 F 3 "" H 9400 4300 50  0000 C CNN
 	1    9400 4300
@@
 $EndComp
 $Comp
-L LED D12
+L LED-RESCUE-np08 D12
 U 1 1 57A4DEA5
 P 9700 4400
+AR Path="/57A4DEA5" Ref="D12"  Part="1"
+AR Path="/57A4D8D4/57A4DEA5" Ref="D12"  Part="1"
 F 0 "D12" H 9700 4500 50  0000 C CNN
 F 1 "LED" H 9700 4300 50  0000 C CNN
-F 2 "LEDs:LED-5MM" H 9700 4400 50  0001 C CNN
+F 2 "" H 9700 4400 50  0001 C CNN
 F 3 "" H 9700 4400 50  0000 C CNN
 	1    9700 4400
@@
 	9500 4400 7400 4400
 $Comp
-L LED D13
+L LED-RESCUE-np08 D13
 U 1 1 57A4E19D
 P 10000 4500
+AR Path="/57A4E19D" Ref="D13"  Part="1"
+AR Path="/57A4D8D4/57A4E19D" Ref="D13"  Part="1"
 F 0 "D13" H 10000 4600 50  0000 C CNN
 F 1 "LED" H 10000 4400 50  0000 C CNN
-F 2 "LEDs:LED-5MM" H 10000 4500 50  0001 C CNN
+F 2 "" H 10000 4500 50  0001 C CNN
 F 3 "" H 10000 4500 50  0000 C CNN
 	1    10000 4500
@@
 F 0 "P16" H 7850 5700 50  0000 C CNN
 F 1 "CONN_01X08" V 7950 5250 50  0000 C CNN
-F 2 "Pin_Headers:Pin_Header_Straight_1x08" H 7850 5250 50  0001 C CNN
+F 2 "" H 7850 5250 50  0001 C CNN
 F 3 "" H 7850 5250 50  0000 C CNN
 	1    7850 5250
@@
 P 3850 5250
 F 0 "P15" H 3850 5700 50  0000 C CNN
-F 1 "CONN_01X08" V 3950 5250 50  0000 C CNN
-F 2 "Pin_Headers:Pin_Header_Straight_1x08" H 3850 5250 50  0001 C CNN
+F 1 "PORTB" V 3950 5250 50  0000 C CNN
+F 2 "Pin_Headers:Pin_Header_Straight_1x08_Pitch1.27mm" H 3850 5250 50  0001 C CNN
 F 3 "" H 3850 5250 50  0000 C CNN
 	1    3850 5250
