File: kicad/alimentacion.sch (KiCad schematic (older format))
At the start: 19 parts, among them P3 aliment., P4 sw_aliment, P5 sw_pic, P6 CONN_01X03, P7 CONN_01X03, U1 LM78L05ACZ, U2 LM7805CT

Commit message: prototipo base para icaro version SMD
Parts:
- C10, C6, C7, C9: footprint Capacitors_ThroughHole:C_Radial_D5_L6_P2.5 -> (none)
- C11, C8: footprint Capacitors_ThroughHole:C_Disc_D3_P2.5 -> (none)
- D2, D4: footprint LEDs:LED-5MM -> (none); symbol LED -> LED-RESCUE-np08
- D3, D5: footprint Diodes_ThroughHole:Diode_DO-35_SOD27_Horizontal_RM10 -> (none)
- P3: footprint Connect:bornier2 -> Pin_Headers:Pin_Header_Straight_1x02_Pitch1.27mm
- P4, P6, P7: footprint Pin_Headers:Pin_Header_Straight_1x03 -> (none)
- P5: footprint Pin_Headers:Pin_Header_Straight_1x03 -> Pin_Headers:Pin_Header_Straight_1x03_Pitch1.27mm
- R3, R4: footprint Resistors_ThroughHole:Resistor_Horizontal_RM15mm -> (none)
- U1: footprint TO_SOT_Packages_THT:TO-92_Molded_Narrow -> (none)
- U2: footprint TO_SOT_Packages_THT:TO-220_Neutral123_Horizontal -> (none)
Connections:
- net VDD: now also P5.2 (P2); no longer P5.1 (P1)
- net vcc_con: no longer P5.2 (P2)
- net uno_estos_dos_para_la_prueba_SMD: now reaches P3.1 (P1), P4.2 (P2)
- net uno_estos_dos_para_la_prueba_SMD: now also P5.3 (P3)
Changed lines of the file:
@@
 EESchema Schematic File Version 2
+LIBS:np08-rescue
 LIBS:power
 LIBS:device
@@
 F 0 "C8" H 6375 3550 50  0000 L CNN
 F 1 "0.1uF" H 6375 3350 50  0000 L CNN
-F 2 "Capacitors_ThroughHole:C_Disc_D3_P2.5" H 6388 3300 50  0001 C CNN
+F 2 "" H 6388 3300 50  0001 C CNN
 F 3 "" H 6350 3450 50  0000 C CNN
 	1    6350 3450
@@
 F 0 "C7" H 5975 3550 50  0000 L CNN
 F 1 "100 uF-electr" H 5650 3250 50  0000 L CNN
-F 2 "Capacitors_ThroughHole:C_Radial_D5_L6_P2.5" H 5988 3300 50  0001 C CNN
+F 2 "" H 5988 3300 50  0001 C CNN
 F 3 "" H 5950 3450 50  0000 C CNN
 	1    5950 3450
@@
 F 0 "C6" H 4625 3550 50  0000 L CNN
 F 1 "100uF-electr" H 4450 3250 50  0000 L CNN
-F 2 "Capacitors_ThroughHole:C_Radial_D5_L6_P2.5" H 4638 3300 50  0001 C CNN
+F 2 "" H 4638 3300 50  0001 C CNN
 F 3 "" H 4600 3450 50  0000 C CNN
 	1    4600 3450
@@
 $EndComp
 $Comp
-L LED D2
+L LED-RESCUE-np08 D2
 U 1 1 579A692B
 P 6700 4000
+AR Path="/579A692B" Ref="D2"  Part="1"
+AR Path="/579A6704/579A692B" Ref="D2"  Part="1"
 F 0 "D2" H 6700 4100 50  0000 C CNN
 F 1 "LED" H 6700 3900 50  0000 C CNN
-F 2 "LEDs:LED-5MM" H 6700 4000 50  0001 C CNN
+F 2 "" H 6700 4000 50  0001 C CNN
 F 3 "" H 6700 4000 50  0000 C CNN
 	1    6700 4000
@@
 F 0 "R3" V 6780 3450 50  0000 C CNN
 F 1 "470" V 6700 3450 50  0000 C CNN
-F 2 "Resistors_ThroughHole:Resistor_Horizontal_RM15mm" V 6630 3450 50  0001 C CNN
+F 2 "" V 6630 3450 50  0001 C CNN
 F 3 "" H 6700 3450 50  0000 C CNN
 	1    6700 3450
@@
 F 0 "P3" H 2550 2650 50  0000 C CNN
 F 1 "aliment." V 2650 2500 50  0000 C CNN
-F 2 "Connect:bornier2" H 2550 2500 50  0001 C CNN
+F 2 "Pin_Headers:Pin_Header_Straight_1x02_Pitch1.27mm" H 2550 2500 50  0001 C CNN
 F 3 "" H 2550 2500 50  0000 C CNN
 	1    2550 2500
@@
 F 0 "U1" H 5050 3550 50  0000 C CNN
 F 1 "LM78L05ACZ" H 5250 3550 50  0000 L CNN
-F 2 "TO_SOT_Packages_THT:TO-92_Molded_Narrow" H 5250 3650 50  0000 C CIN
+F 2 "" H 5250 3650 50  0001 C CIN
 F 3 "" H 5250 3350 50  0000 C CNN
 	1    5250 3350
@@
 F 0 "U2" H 5050 2250 50  0000 C CNN
 F 1 "LM7805CT" H 5250 2250 50  0000 L CNN
-F 2 "TO_SOT_Packages_THT:TO-220_Neutral123_Horizontal" H 5250 2400 50  0000 C CIN
+F 2 "" H 5250 2400 50  0001 C CIN
 F 3 "" H 5250 2050 50  0000 C CNN
 	1    5250 2050
@@
 F 0 "C9" H 4475 2250 50  0000 L CNN
 F 1 "100uF-electr" H 4550 2000 50  0000 L CNN
-F 2 "Capacitors_ThroughHole:C_Radial_D5_L6_P2.5" H 4488 2000 50  0001 C CNN
+F 2 "" H 4488 2000 50  0001 C CNN
 F 3 "" H 4450 2150 50  0000 C CNN
 	1    4450 2150
@@
 F 0 "C10" H 5925 2250 50  0000 L CNN
 F 1 "100 uF-electr" H 5850 2450 50  0000 L CNN
-F 2 "Capacitors_ThroughHole:C_Radial_D5_L6_P2.5" H 5938 2000 50  0001 C CNN
+F 2 "" H 5938 2000 50  0001 C CNN
 F 3 "" H 5900 2150 50  0000 C CNN
 	1    5900 2150
@@
 F 0 "C11" H 6475 2250 50  0000 L CNN
 F 1 "0.1uF" H 6475 2050 50  0000 L CNN
-F 2 "Capacitors_ThroughHole:C_Disc_D3_P2.5" H 6488 2000 50  0001 C CNN
+F 2 "" H 6488 2000 50  0001 C CNN
 F 3 "" H 6450 2150 50  0000 C CNN
 	1    6450 2150
@@
 F 0 "R4" V 6980 2150 50  0000 C CNN
 F 1 "470" V 6900 2150 50  0000 C CNN
-F 2 "Resistors_ThroughHole:Resistor_Horizontal_RM15mm" V 6830 2150 50  0001 C CNN
+F 2 "" V 6830 2150 50  0001 C CNN
 F 3 "" H 6900 2150 50  0000 C CNN
 	1    6900 2150
@@
 $EndComp
 $Comp
-L LED D4
+L LED-RESCUE-np08 D4
 U 1 1 579B97B7
 P 6900 2650
+AR Path="/579B97B7" Ref="D4"  Part="1"
+AR Path="/579A6704/579B97B7" Ref="D4"  Part="1"
 F 0 "D4" H 6900 2750 50  0000 C CNN
 F 1 "LED" H 6900 2550 50  0000 C CNN
-F 2 "LEDs:LED-5MM" H 6900 2650 50  0001 C CNN
+F 2 "" H 6900 2650 50  0001 C CNN
 F 3 "" H 6900 2650 50  0000 C CNN
 	1    6900 2650
@@
 F 0 "P4" H 2150 3500 50  0000 C CNN
 F 1 "sw_aliment" V 2250 3300 50  0000 C CNN
-F 2 "Pin_Headers:Pin_Header_Straight_1x03" H 2150 3300 50  0001 C CNN
+F 2 "" H 2150 3300 50  0001 C CNN
 F 3 "" H 2150 3300 50  0000 C CNN
 	1    2150 3300
@@
 F 0 "D3" H 2500 4050 50  0000 C CNN
 F 1 "D" H 2500 3850 50  0000 C CNN
-F 2 "Diodes_ThroughHole:Diode_DO-35_SOD27_Horizontal_RM10" H 2500 3950 50  0001 C CNN
+F 2 "" H 2500 3950 50  0001 C CNN
 F 3 "" H 2500 3950 50  0000 C CNN
 	1    2500 3950
@@
 F 0 "P7" H 7800 3550 50  0000 C CNN
 F 1 "CONN_01X03" V 7900 3350 50  0000 C CNN
-F 2 "Pin_Headers:Pin_Header_Straight_1x03" H 7800 3350 50  0001 C CNN
+F 2 "" H 7800 3350 50  0001 C CNN
 F 3 "" H 7800 3350 50  0000 C CNN
 	1    7800 3350
@@
 F 0 "P5" H 2800 3500 50  0000 C CNN
 F 1 "sw_pic" V 2900 3300 50  0000 C CNN
-F 2 "Pin_Headers:Pin_Header_Straight_1x03" H 2800 3300 50  0001 C CNN
+F 2 "Pin_Headers:Pin_Header_Straight_1x03_Pitch1.27mm" H 2800 3300 50  0001 C CNN
 F 3 "" H 2800 3300 50  0000 C CNN
 	1    2800 3300
@@
 $EndComp
 Wire Wire Line
-	3000 3400 3100 3400
-Wire Wire Line
-	3100 3400 3100 3900
+	3100 3300 3100 3900
 Text GLabel 7800 3700 3    60   Input ~ 0
 vcc_con
@@
 vcc_con
 Wire Wire Line
-	3000 3300 3050 3300
-Wire Wire Line
-	3050 3300 3050 3000
+	3000 3300 3100 3300
 Wire Wire Line
 	7800 3700 7800 3550
@@
 F 0 "D5" H 7800 3100 50  0000 C CNN
 F 1 "D" H 7800 2900 50  0000 C CNN
-F 2 "Diodes_ThroughHole:Diode_DO-35_SOD27_Horizontal_RM10" H 7800 3000 50  0001 C CNN
+F 2 "" H 7800 3000 50  0001 C CNN
 F 3 "" H 7800 3000 50  0000 C CNN
 	1    7800 3000
@@
 F 0 "P6" H 7350 1200 50  0000 C CNN
 F 1 "CONN_01X03" V 7450 1000 50  0000 C CNN
-F 2 "Pin_Headers:Pin_Header_Straight_1x03" H 7350 1000 50  0001 C CNN
+F 2 "" H 7350 1000 50  0001 C CNN
 F 3 "" H 7350 1000 50  0000 C CNN
 	1    7350 1000
@@
 Wire Wire Line
 	8200 2200 8200 3000
+Wire Wire Line
+	2500 3100 3000 3100
+Wire Wire Line
+	3000 3100 3000 3200
+Connection ~ 2500 3100
+Text Label 2800 3100 1    60   ~ 0
+uno_estos_dos_para_la_prueba_SMD
 $EndSCHEMATC
