File: kicad/motores_cc.sch (KiCad schematic (older format))
At the start: 4 parts, among them P8 CONN_01X02, P9 CONN_01X02, U3 L293D

Commit message: prototipo base para icaro version SMD
Parts:
- C12: footprint Capacitors_ThroughHole:C_Disc_D3_P2.5 -> (none)
- P8, P9: footprint Connect:bornier2 -> (none)
- U3: footprint Housings_DIP:DIP-16_W7.62mm -> (none)
Changed lines of the file:
@@
 EESchema Schematic File Version 2
+LIBS:np08-rescue
 LIBS:power
 LIBS:device
@@
 F 0 "U3" H 4950 3150 60  0000 C CNN
 F 1 "L293D" H 5600 3150 60  0000 C CNN
-F 2 "Housings_DIP:DIP-16_W7.62mm" H 5250 2550 60  0001 C CNN
+F 2 "" H 5250 2550 60  0001 C CNN
 F 3 "" H 5250 2550 60  0000 C CNN
 	1    5250 2550
@@
 F 0 "P9" H 7350 1800 50  0000 C CNN
 F 1 "CONN_01X02" V 7450 1650 50  0000 C CNN
-F 2 "Connect:bornier2" H 7350 1650 50  0001 C CNN
+F 2 "" H 7350 1650 50  0001 C CNN
 F 3 "" H 7350 1650 50  0000 C CNN
 	1    7350 1650
@@
 F 0 "P8" H 4200 1800 50  0000 C CNN
 F 1 "CONN_01X02" V 4300 1650 50  0000 C CNN
-F 2 "Connect:bornier2" H 4200 1650 50  0001 C CNN
+F 2 "" H 4200 1650 50  0001 C CNN
 F 3 "" H 4200 1650 50  0000 C CNN
 	1    4200 1650
@@
 F 0 "C12" H 4875 3750 50  0000 L CNN
 F 1 "0.1uF" H 4875 3550 50  0000 L CNN
-F 2 "Capacitors_ThroughHole:C_Disc_D3_P2.5" H 4888 3500 50  0001 C CNN
+F 2 "" H 4888 3500 50  0001 C CNN
 F 3 "" H 4850 3650 50  0000 C CNN
 	1    4850 3650
