File: kicad/motores_cc.sch (KiCad schematic (older format))
At the start: 4 parts, among them P8 CONN_01X02, P9 CONN_01X02, U3 L293D

Commit message: cambios en la placa np08
Parts:
- C12: footprint Capacitors_ThroughHole:C_Disc_D3_P2.5 -> Capacitors_THT:C_Disc_D3.4mm_W2.1mm_P2.50mm
- P8: value CONN_01X02 -> MOTOR_2; footprint Connect:bornier2 -> Connectors:bornier2
- P9: value CONN_01X02 -> MOTOR_1; footprint Connect:bornier2 -> Connectors:bornier2
- U3: footprint Housings_DIP:DIP-16_W7.62mm -> Housings_DIP:DIP-16_W7.62mm_LongPads
Connections:
- net at U3.11 (OUPUT_3): now also P9.2 (P2); no longer P8.1 (P1)
- net at U3.6 (OUPUT_2): now also P8.1 (P1); no longer P9.2 (P2)
Changed lines of the file:
@@
 F 0 "U3" H 4950 3150 60  0000 C CNN
 F 1 "L293D" H 5600 3150 60  0000 C CNN
-F 2 "Housings_DIP:DIP-16_W7.62mm" H 5250 2550 60  0001 C CNN
+F 2 "Housings_DIP:DIP-16_W7.62mm_LongPads" H 5250 2550 60  0001 C CNN
 F 3 "" H 5250 2550 60  0000 C CNN
 	1    5250 2550
@@
 P 7350 1650
 F 0 "P9" H 7350 1800 50  0000 C CNN
-F 1 "CONN_01X02" V 7450 1650 50  0000 C CNN
-F 2 "Connect:bornier2" H 7350 1650 50  0001 C CNN
+F 1 "MOTOR_1" V 7450 1650 50  0000 C CNN
+F 2 "Connectors:bornier2" H 7350 1650 50  0001 C CNN
 F 3 "" H 7350 1650 50  0000 C CNN
 	1    7350 1650
@@
 P 4200 1650
 F 0 "P8" H 4200 1800 50  0000 C CNN
-F 1 "CONN_01X02" V 4300 1650 50  0000 C CNN
-F 2 "Connect:bornier2" H 4200 1650 50  0001 C CNN
+F 1 "MOTOR_2" V 4300 1650 50  0000 C CNN
+F 2 "Connectors:bornier2" H 4200 1650 50  0001 C CNN
 F 3 "" H 4200 1650 50  0000 C CNN
 	1    4200 1650
@@
 $EndComp
 Wire Wire Line
-	6050 2350 7300 2350
-Wire Wire Line
-	7300 2350 7300 1850
-Wire Wire Line
 	4550 2350 4250 2350
 Wire Wire Line
 	4250 2350 4250 1850
-Wire Wire Line
-	4150 1850 4150 3250
-Wire Wire Line
-	4150 3250 6650 3250
-Wire Wire Line
-	6650 3250 6650 2800
-Wire Wire Line
-	6650 2800 6050 2800
-Wire Wire Line
-	7400 1850 7400 3450
-Wire Wire Line
-	7400 3450 4250 3450
-Wire Wire Line
-	4250 3450 4250 2800
-Wire Wire Line
-	4250 2800 4550 2800
 Wire Wire Line
 	6050 2650 6050 2500
@@
 	4550 2650 4550 2500
 $Comp
-L GND #PWR019
+L GND #PWR030
 U 1 1 579BDCF1
 P 6150 2550
-F 0 "#PWR019" H 6150 2300 50  0001 C CNN
+F 0 "#PWR030" H 6150 2300 50  0001 C CNN
 F 1 "GND" H 6150 2400 50  0000 C CNN
 F 2 "" H 6150 2550 50  0000 C CNN
@@
 $EndComp
 $Comp
-L GND #PWR020
+L GND #PWR031
 U 1 1 579BDD17
 P 4450 2550
-F 0 "#PWR020" H 4450 2300 50  0001 C CNN
+F 0 "#PWR031" H 4450 2300 50  0001 C CNN
 F 1 "GND" H 4450 2400 50  0000 C CNN
 F 2 "" H 4450 2550 50  0000 C CNN
@@
 input4
 Wire Wire Line
-	6050 2200 6750 2200
-Wire Wire Line
 	6750 2950 6050 2950
 Wire Wire Line
 	4550 2950 4000 2950
-Wire Wire Line
-	3950 2200 4550 2200
 $Comp
 L C C12
@@
 F 0 "C12" H 4875 3750 50  0000 L CNN
 F 1 "0.1uF" H 4875 3550 50  0000 L CNN
-F 2 "Capacitors_ThroughHole:C_Disc_D3_P2.5" H 4888 3500 50  0001 C CNN
+F 2 "Capacitors_THT:C_Disc_D3.4mm_W2.1mm_P2.50mm" H 4888 3500 50  0001 C CNN
 F 3 "" H 4850 3650 50  0000 C CNN
 	1    4850 3650
@@
 Connection ~ 4650 3300
 $Comp
-L GND #PWR021
+L GND #PWR032
 U 1 1 579F6E96
 P 5150 3750
-F 0 "#PWR021" H 5150 3500 50  0001 C CNN
+F 0 "#PWR032" H 5150 3500 50  0001 C CNN
 F 1 "GND" H 5150 3600 50  0000 C CNN
 F 2 "" H 5150 3750 50  0000 C CNN
@@
 Wire Wire Line
 	5150 3650 5150 3750
+Wire Wire Line
+	4550 2800 4150 2800
+Wire Wire Line
+	4150 2800 4150 1850
+Wire Wire Line
+	6050 2350 7300 2350
+Wire Wire Line
+	7300 2350 7300 1850
+Wire Wire Line
+	7400 1850 7400 2800
+Wire Wire Line
+	7400 2800 6050 2800
+Wire Wire Line
+	6050 2200 6750 2200
+Wire Wire Line
+	3950 2200 4550 2200
 $EndSCHEMATC

Commit message: cambios para el desarrollo de la placa np08, ahora usa 6 pines para servos y 3 pines para dig
Connections:
- net at U3.11 (OUPUT_3): now also P8.1 (P1); no longer P9.2 (P2)
- net at U3.14 (OUPUT_4): now also P9.2 (P2); no longer P9.1 (P1)
- net at U3.6 (OUPUT_2): now also P9.1 (P1); no longer P8.1 (P1)
Other:
- moved on the sheet: P9
Changed lines of the file:
@@
 L CONN_01X02 P9
 U 1 1 579BDA17
-P 7350 1650
-F 0 "P9" H 7350 1800 50  0000 C CNN
-F 1 "MOTOR_1" V 7450 1650 50  0000 C CNN
-F 2 "Connectors:bornier2" H 7350 1650 50  0001 C CNN
-F 3 "" H 7350 1650 50  0000 C CNN
-	1    7350 1650
-	0    -1   -1   0
+P 7800 2200
+F 0 "P9" H 7800 2350 50  0000 C CNN
+F 1 "MOTOR_1" V 7900 2200 50  0000 C CNN
+F 2 "Connectors:bornier2" H 7800 2200 50  0001 C CNN
+F 3 "" H 7800 2200 50  0000 C CNN
+	1    7800 2200
+	1    0    0    -1
 $EndComp
 $Comp
@@
 	5150 3650 5150 3750
 Wire Wire Line
-	4550 2800 4150 2800
-Wire Wire Line
-	4150 2800 4150 1850
-Wire Wire Line
-	6050 2350 7300 2350
-Wire Wire Line
-	7300 2350 7300 1850
-Wire Wire Line
-	7400 1850 7400 2800
-Wire Wire Line
-	7400 2800 6050 2800
-Wire Wire Line
 	6050 2200 6750 2200
 Wire Wire Line
 	3950 2200 4550 2200
+Wire Wire Line
+	4150 1850 4150 3450
+Wire Wire Line
+	4150 3450 7200 3450
+Wire Wire Line
+	7200 3450 7200 2800
+Wire Wire Line
+	7200 2800 6050 2800
+Wire Wire Line
+	4550 2800 4350 2800
+Wire Wire Line
+	4350 2800 4350 4050
+Wire Wire Line
+	4350 4050 8050 4050
+Wire Wire Line
+	6050 2350 7350 2350
+Wire Wire Line
+	7350 2350 7350 2250
+Wire Wire Line
+	7350 2250 7600 2250
+Wire Wire Line
+	7600 2150 7600 1900
+Wire Wire Line
+	7600 1900 8050 1900
+Wire Wire Line
+	8050 1900 8050 4050
 $EndSCHEMATC
