File: kicad/np08.sch (KiCad schematic (older format))
At the start: 18 parts, among them P1 USB_B, P10 CONN_01X02, P11 CONN_01X02, P12 analog, P13 GND, P14 +5V, P2 CONN_01X04, SW1 SW_PUSH, Y1 Crystal

Commit message: prototipo base para icaro version SMD
Parts:
- added J1: RC0-RC1-RC2, Pin_Headers:Pin_Header_Straight_1x03_Pitch1.27mm, symbol CONN_01X03
- added P17: RX-TX, Pin_Headers:Pin_Header_Straight_1x02_Pitch1.27mm, symbol CONN_01X02
- C1: footprint Capacitors_ThroughHole:C_Radial_D5_L6_P2.5 -> Capacitors_SMD:CP_Elec_3x5.3
- C2: footprint Capacitors_ThroughHole:C_Disc_D3_P2.5 -> (none)
- C3, C4, C5: footprint Capacitors_ThroughHole:C_Disc_D3_P2.5 -> Capacitors_SMD:C_0603_HandSoldering
- D1: footprint LEDs:LED-5MM -> LEDs:LED_0805; symbol LED -> LED-RESCUE-np08
- P1: footprint Connect:USB_B -> w_conn_pc:conn_usb_B_micro_smd; symbol USB_B -> USB_B-RESCUE-np08
- P10, P11: footprint Pin_Headers:Pin_Header_Straight_1x02 -> Pin_Headers:Pin_Header_Straight_1x02_Pitch1.27mm
- P12: footprint Pin_Headers:Pin_Header_Straight_1x08 -> Pin_Headers:Pin_Header_Straight_1x08_Pitch1.27mm
- P13, P14: footprint Pin_Headers:Pin_Header_Straight_1x08 -> (none)
- P2: footprint Pin_Headers:Pin_Header_Straight_1x04 -> Pin_Headers:Pin_Header_Straight_1x04_Pitch1.27mm
- R1, R2: footprint Resistors_ThroughHole:Resistor_Horizontal_RM15mm -> Resistors_SMD:R_0603
- SW1: footprint Buttons_Switches_ThroughHole:SW_PUSH-12mm -> Buttons_Switches_SMD:SW_SPST_EVQP0
- U***1: footprint Housings_DIP:DIP-40_W15.24mm -> Housings_QFP:LQFP-44_10x10mm_Pitch0.8mm
- Y1: footprint Crystals:Crystal_HC50-U_Vertical -> Crystals:Crystal_SMD_HC49-SD
Connections:
- net labels added: RC0, RC1, RC2, RC6, RC7
- wire segments 103 -> 108
Changed lines of the file:
@@
 EESchema Schematic File Version 2
+LIBS:np08-rescue
 LIBS:power
 LIBS:device
@@
 F 0 "U***1" H 6500 3850 70  0000 C CNN
 F 1 "PIC18F4550" H 6500 3650 70  0000 C CNN
-F 2 "Housings_DIP:DIP-40_W15.24mm" H 6500 3750 60  0001 C CNN
+F 2 "Housings_QFP:LQFP-44_10x10mm_Pitch0.8mm" H 6500 3750 60  0001 C CNN
 F 3 "" H 6500 3750 60  0000 C CNN
 	1    6500 3750
@@
 F 0 "SW1" H 4300 3110 50  0000 C CNN
 F 1 "SW_PUSH" H 4150 2920 50  0000 C CNN
-F 2 "Buttons_Switches_ThroughHole:SW_PUSH-12mm" H 4150 3000 50  0001 C CNN
+F 2 "Buttons_Switches_SMD:SW_SPST_EVQP0" H 4150 3000 50  0001 C CNN
 F 3 "" H 4150 3000 50  0000 C CNN
 	1    4150 3000
@@
 F 0 "C1" H 3775 3100 50  0000 L CNN
 F 1 "10 uF-electr" V 3900 2800 50  0000 L CNN
-F 2 "Capacitors_ThroughHole:C_Radial_D5_L6_P2.5" H 3788 2850 50  0001 C CNN
+F 2 "Capacitors_SMD:CP_Elec_3x5.3" H 3788 2850 50  0001 C CNN
 F 3 "" H 3750 3000 50  0000 C CNN
 	1    3750 3000
@@
 F 0 "R2" V 3830 2400 50  0000 C CNN
 F 1 "1K" V 3750 2400 50  0000 C CNN
-F 2 "Resistors_ThroughHole:Resistor_Horizontal_RM15mm" V 3680 2400 50  0001 C CNN
+F 2 "Resistors_SMD:R_0603" V 3680 2400 50  0001 C CNN
 F 3 "" H 3750 2400 50  0000 C CNN
 	1    3750 2400
@@
 F 0 "R1" V 3530 2950 50  0000 C CNN
 F 1 "470" V 3450 2950 50  0000 C CNN
-F 2 "Resistors_ThroughHole:Resistor_Horizontal_RM15mm" V 3380 2950 50  0001 C CNN
+F 2 "Resistors_SMD:R_0603" V 3380 2950 50  0001 C CNN
 F 3 "" H 3450 2950 50  0000 C CNN
 	1    3450 2950
@@
 $EndComp
 $Comp
-L LED D1
+L LED-RESCUE-np08 D1
 U 1 1 579A397D
 P 3450 2450
 F 0 "D1" H 3450 2550 50  0000 C CNN
 F 1 "LED" H 3450 2350 50  0000 C CNN
-F 2 "LEDs:LED-5MM" H 3450 2450 50  0001 C CNN
+F 2 "LEDs:LED_0805" H 3450 2450 50  0001 C CNN
 F 3 "" H 3450 2450 50  0000 C CNN
 	1    3450 2450
@@
 F 0 "C2" H 4225 3800 50  0000 L CNN
 F 1 "C" H 4225 3600 50  0000 L CNN
-F 2 "Capacitors_ThroughHole:C_Disc_D3_P2.5" H 4238 3550 50  0001 C CNN
+F 2 "" H 4238 3550 50  0001 C CNN
 F 3 "" H 4200 3700 50  0000 C CNN
 	1    4200 3700
@@
 F 0 "C5" H 4975 4600 50  0000 L CNN
 F 1 "220nF" H 4975 4400 50  0000 L CNN
-F 2 "Capacitors_ThroughHole:C_Disc_D3_P2.5" H 4988 4350 50  0001 C CNN
+F 2 "Capacitors_SMD:C_0603_HandSoldering" H 4988 4350 50  0001 C CNN
 F 3 "" H 4950 4500 50  0000 C CNN
 	1    4950 4500
@@
 F 0 "Y1" H 4800 4250 50  0000 C CNN
 F 1 "Crystal" H 4800 3950 50  0000 C CNN
-F 2 "Crystals:Crystal_HC50-U_Vertical" H 4800 4100 50  0001 C CNN
+F 2 "Crystals:Crystal_SMD_HC49-SD" H 4800 4100 50  0001 C CNN
 F 3 "" H 4800 4100 50  0000 C CNN
 	1    4800 4100
@@
 F 0 "C4" H 4525 4550 50  0000 L CNN
 F 1 "22pF" H 4525 4350 50  0000 L CNN
-F 2 "Capacitors_ThroughHole:C_Disc_D3_P2.5" H 4538 4300 50  0001 C CNN
+F 2 "Capacitors_SMD:C_0603_HandSoldering" H 4538 4300 50  0001 C CNN
 F 3 "" H 4500 4450 50  0000 C CNN
 	1    4500 4450
@@
 F 0 "C3" H 4225 4550 50  0000 L CNN
 F 1 "22pF" H 4225 4350 50  0000 L CNN
-F 2 "Capacitors_ThroughHole:C_Disc_D3_P2.5" H 4238 4300 50  0001 C CNN
+F 2 "Capacitors_SMD:C_0603_HandSoldering" H 4238 4300 50  0001 C CNN
 F 3 "" H 4200 4450 50  0000 C CNN
 	1    4200 4450
@@
 	7550 3300 7650 3300
 $Comp
-L USB_B P1
+L USB_B-RESCUE-np08 P1
 U 1 1 579A4922
 P 2950 4650
 F 0 "P1" H 3150 4450 50  0000 C CNN
 F 1 "USB_B" H 2900 4850 50  0000 C CNN
-F 2 "Connect:USB_B" V 2900 4550 50  0001 C CNN
+F 2 "w_conn_pc:conn_usb_B_micro_smd" V 2900 4550 50  0001 C CNN
 F 3 "" V 2900 4550 50  0000 C CNN
 	1    2950 4650
@@
 F 0 "P10" H 8700 5650 50  0000 C CNN
 F 1 "CONN_01X02" V 8800 5500 50  0000 C CNN
-F 2 "Pin_Headers:Pin_Header_Straight_1x02" H 8700 5500 50  0001 C CNN
+F 2 "Pin_Headers:Pin_Header_Straight_1x02_Pitch1.27mm" H 8700 5500 50  0001 C CNN
 F 3 "" H 8700 5500 50  0000 C CNN
 	1    8700 5500
@@
 F 0 "P11" H 8700 5150 50  0000 C CNN
 F 1 "CONN_01X02" V 8800 5000 50  0000 C CNN
-F 2 "Pin_Headers:Pin_Header_Straight_1x02" H 8700 5000 50  0001 C CNN
+F 2 "Pin_Headers:Pin_Header_Straight_1x02_Pitch1.27mm" H 8700 5000 50  0001 C CNN
 F 3 "" H 8700 5000 50  0000 C CNN
 	1    8700 5000
@@
 F 0 "P2" H 8700 4700 50  0000 C CNN
 F 1 "CONN_01X04" V 8800 4450 50  0000 C CNN
-F 2 "Pin_Headers:Pin_Header_Straight_1x04" H 8700 4450 50  0001 C CNN
+F 2 "Pin_Headers:Pin_Header_Straight_1x04_Pitch1.27mm" H 8700 4450 50  0001 C CNN
 F 3 "" H 8700 4450 50  0000 C CNN
 	1    8700 4450
@@
 F 0 "P12" H 4800 3300 50  0000 C CNN
 F 1 "analog" V 4900 2850 50  0000 C CNN
-F 2 "Pin_Headers:Pin_Header_Straight_1x08" H 4800 2850 50  0001 C CNN
+F 2 "Pin_Headers:Pin_Header_Straight_1x08_Pitch1.27mm" H 4800 2850 50  0001 C CNN
 F 3 "" H 4800 2850 50  0000 C CNN
 	1    4800 2850
@@
 F 0 "P14" H 9200 1300 50  0000 C CNN
 F 1 "+5V" V 9300 850 50  0000 C CNN
-F 2 "Pin_Headers:Pin_Header_Straight_1x08" H 9200 850 50  0001 C CNN
+F 2 "" H 9200 850 50  0001 C CNN
 F 3 "" H 9200 850 50  0000 C CNN
 	1    9200 850
@@
 F 0 "P13" H 8250 1300 50  0000 C CNN
 F 1 "GND" V 8350 850 50  0000 C CNN
-F 2 "Pin_Headers:Pin_Header_Straight_1x08" H 8250 850 50  0001 C CNN
+F 2 "" H 8250 850 50  0001 C CNN
 F 3 "" H 8250 850 50  0000 C CNN
 	1    8250 850
@@
 	9350 3200 10250 3200
 Connection ~ 10000 1850
+Text GLabel 5250 4300 0    60   Input ~ 0
+RC1
+Text GLabel 5450 4400 0    60   Input ~ 0
+RC2
+Text GLabel 5450 4200 0    60   Input ~ 0
+RC0
+Wire Wire Line
+	5250 4300 5450 4300
+Text GLabel 5450 4800 0    60   Input ~ 0
+RC6
+Text GLabel 5200 4900 0    60   Input ~ 0
+RC7
+Wire Wire Line
+	5200 4900 5450 4900
+Text GLabel 4400 5550 0    60   Input ~ 0
+RC0
+Text GLabel 4650 5650 0    60   Input ~ 0
+RC1
+Text GLabel 4400 5750 0    60   Input ~ 0
+RC2
+Text GLabel 4650 6150 0    60   Input ~ 0
+RC6
+Text GLabel 4400 6250 0    60   Input ~ 0
+RC7
+$Comp
+L CONN_01X02 P17
+U 1 1 5924EF4B
+P 4850 6200
+F 0 "P17" H 4850 6350 50  0000 C CNN
+F 1 "RX-TX" V 4950 6200 50  0000 C CNN
+F 2 "Pin_Headers:Pin_Header_Straight_1x02_Pitch1.27mm" H 4850 6200 50  0001 C CNN
+F 3 "" H 4850 6200 50  0000 C CNN
+	1    4850 6200
+	1    0    0    -1
+$EndComp
+Wire Wire Line
+	4400 6250 4650 6250
+$Comp
+L CONN_01X03 J1
+U 1 1 5924F188
+P 4850 5650
+F 0 "J1" H 4850 5850 50  0000 C CNN
+F 1 "RC0-RC1-RC2" V 4950 5650 50  0000 C CNN
+F 2 "Pin_Headers:Pin_Header_Straight_1x03_Pitch1.27mm" H 4850 5650 50  0001 C CNN
+F 3 "" H 4850 5650 50  0001 C CNN
+	1    4850 5650
+	1    0    0    -1
+$EndComp
+Wire Wire Line
+	4400 5550 4650 5550
+Wire Wire Line
+	4650 5750 4400 5750
 $EndSCHEMATC
